File: SY99_8MBEX.kicad_pcb (KiCad board)
At the start: 2 copper layers, 69 x 100 mm, 30 parts, among them J1 Conn_01x02, J2 Conn_02x20_Odd_Even, J3 Conn_01x14, J4 Conn_02x20_Odd_Even, U1 74ALVC164245DGG,51, U10 TXB0108PWR, U2 74ALVC164245DGG,51, U3 AZ1117EH-3.3TRG1, U4 SN74LVC1G97DBVR, U5 SN74LVC1G97DBVR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

Commit message: Version 1.1
Parts:
- removed U10: TXB0108PWR, TXB0108PWR:TSSOP20
- added C11: 100n, Capacitors_SMD:C_0805_HandSoldering, B.Cu at (159.6, 86.2)
- added C12: 100n, Capacitors_SMD:C_0805_HandSoldering, B.Cu at (151.0, 86.5)
- added C13: 100n, Capacitors_SMD:C_0805_HandSoldering, B.Cu at (159.6, 77.7)
- added C14: 100n, Capacitors_SMD:C_0805_HandSoldering, B.Cu at (151.0, 77.7)
- added C15: 100n, Capacitors_SMD:C_0805_HandSoldering, B.Cu at (158.5, 56.8)
- added C16: 100n, Capacitors_SMD:C_0805_HandSoldering, B.Cu at (151.0, 56.8)
- added C17: 100n, Capacitors_SMD:C_0805_HandSoldering, B.Cu at (158.5, 63.8)
- added C18: 100n, Capacitors_SMD:C_0805_HandSoldering, B.Cu at (151.1, 63.8)
- added R3: 3k3, Resistors_SMD:R_0805_HandSoldering, F.Cu at (123.5, 99.8)
- added TP1: VRAM, Connectors:PINTST, F.Cu at (109.3, 104.5)
- added TP2: ~IC, Connectors:PINTST, F.Cu at (149.1, 129.0)
- added TP3: ~OE, Connectors:PINTST, F.Cu at (149.1, 131.5)
- added TP4: MSBW, Connectors:PINTST, F.Cu at (149.1, 134.0)
- added TP5: LSBW, Connectors:PINTST, F.Cu at (149.1, 136.6)
- C1, C2, C3: footprint Capacitors_Tantalum_SMD:CP_Tantalum_Case-B_EIA-3528-21_Reflow -> Capacitors_Tantalum_SMD:CP_Tantalum_Case-A_EIA-3216-18_Reflow
- C10, C6, C8, C9: value 0.1u -> 100n; moved to B.Cu
- C7: value 0.1u -> 100n
- D1, D2: footprint digikey-footprints:LED_5mm_Radial -> LEDs:LED_D5.0mm
- J2: footprint Pin_Headers:Pin_Header_Straight_2x20_Pitch2.54mm_SMD -> SY99:Socket_Strip_Straight_2x20_Pitch2.54mm_10.30Wide_SMD; moved to B.Cu
- J3: value Conn_01x14 -> Conn_01x12_Male; footprint Pin_Headers:Pin_Header_Straight_1x14_Pitch2.54mm -> Pin_Headers:Pin_Header_Straight_1x12_Pitch2.54mm
- J4: footprint SY99:Socket_Strip_Straight_2x20_Pitch2.54mm_10.30Wide_SMD -> SY99:Pin_Header_Straight_2x20_Pitch2.54mm_10.30Wide_SMD; moved to F.Cu
- R1: value 220R -> 1K; footprint Resistors_SMD:R_1210_HandSoldering -> Resistors_SMD:R_0805_HandSoldering
- R2: value 150R -> 1K; footprint Resistors_SMD:R_1210_HandSoldering -> Resistors_SMD:R_0805_HandSoldering
- U9: value TXB0108PWR -> SN74LVCH16T245; footprint TXB0108PWR:TSSOP20 -> SN74LVCH16T245:TSSOP48
- moved C9 53.1 mm to (159.5, 102.8), turned to 270 degrees
- moved C6 47.0 mm to (159.5, 93.9), turned to 90 degrees
- moved C8 33.8 mm to (151.0, 94.0), turned to 90 degrees
- moved C7 17.6 mm to (133.2, 52.0)
- moved C10 13.9 mm to (151.0, 103.2), turned to 270 degrees
- moved U9 11.0 mm to (149.8, 54.2)
- moved D1 2.57 mm to (124.3, 106.1)
- moved D2 2.57 mm to (124.3, 117.0)
- moved C4 0.69 mm to (158.9, 70.3)
- moved R2 0.68 mm to (142.3, 119.0)
- moved G*** 0.50 mm to (115.5, 112.0), turned to 90 degrees
- moved J3 0.18 mm to (153.5, 111.2)
- moved J4 0.18 mm to (170.1, 73.9), turned to 0 degrees
- moved J2 0.12 mm to (170.1, 73.9), turned to 180 degrees
Connections:
- C10 pad 1: +5V -> +3V3
- C6 pad 1: +3V3 -> +5V
- C7 pad 1: GND -> /VRAM
- C7 pad 2: +3V3 -> GND
- C8 pad 1: GND -> +3V3
- C8 pad 2: +5V -> GND
- J2 pad 19: Net-(J2-Pad19) -> /AIN23
- J2 pad 20: /AIN23 -> /CST
- J3 pad 10: /~ICIN -> /~MSBWIN
- J3 pad 11: /~OEIN -> /~LSBWIN
- J3 pad 12: /~MSBWIN -> GND
- J3 pad 8: Net-(J3-Pad8) -> /~ICIN
- J3 pad 9: Net-(J3-Pad9) -> /~OEIN
- J4 pad 19: Net-(J4-Pad19) -> /AIN23
- J4 pad 20: /AIN23 -> /CST
- U2 pad 11: Net-(U2-Pad11) -> GND
- U2 pad 19: Net-(U2-Pad19) -> GND
- U2 pad 20: Net-(U2-Pad20) -> GND
- U2 pad 22: Net-(U2-Pad22) -> GND
- U2 pad 23: Net-(U2-Pad23) -> GND
- U2 pad 26: Net-(U2-Pad26) -> GND
- U2 pad 27: Net-(U2-Pad27) -> GND
- U2 pad 29: Net-(U2-Pad29) -> GND
- U2 pad 30: Net-(U2-Pad30) -> GND
- U2 pad 38: Net-(U2-Pad38) -> GND
- U9 pad 1: /DQ7 -> /~OEIN
- U9 pad 10: +3V3 -> GND
- U9 pad 11: GND -> /DQ9
- U9 pad 12: /D0 -> /DQ8
- U9 pad 13: /D1 -> /DQ7
- U9 pad 14: /D2 -> /DQ6
- U9 pad 15: /D3 -> GND
- U9 pad 16: /D4 -> /DQ5
- U9 pad 17: /D5 -> /DQ4
- U9 pad 18: /D6 -> +3V3
- U9 pad 19: +5V -> /DQ3
- U9 pad 2: +3V3 -> /DQ15
- U9 pad 20: /D7 -> /DQ2
- U9 pad 3: /DQ6 -> /DQ14
- U9 pad 4: /DQ5 -> GND
- U9 pad 5: /DQ4 -> /DQ13
- U9 pad 6: /DQ3 -> /DQ12
- U9 pad 7: /DQ2 -> +3V3
- U9 pad 8: /DQ1 -> /DQ11
- U9 pad 9: /DQ0 -> /DQ10
Routing:
- net /~OEIN: track 65.7 -> 93.4 mm, vias 1 -> 4
- net +3V3: track 256.9 -> 234.7 mm, vias 16 -> 15
- net +5V: track 134.6 -> 114.4 mm, vias 7 -> 8
- net /AIN23: track 22.4 -> 38.2 mm, vias 3 -> 4
- net GND: track 563.5 -> 549.3 mm
- net /VRAM: track 97.0 -> 106.6 mm
- net /D7: track 17.2 -> 9.52 mm
- net /D5: track 16.8 -> 9.09 mm
- net /D3: track 16.3 -> 9.52 mm
- net /D9: track 16.6 -> 10.2 mm
- net /D1: track 16.3 -> 9.95 mm
- net /~LSBWIN: track 79.0 -> 72.7 mm
- net /D8: track 22.8 -> 16.6 mm
- net /D6: track 22.1 -> 16.0 mm
- net /~MSBWIN: track 75.5 -> 69.5 mm
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Other:
- board text added: "S/N"
- board text added: "Yamaha SY99 8MB Expansion v1.1 ©2018 Wohmart.COM CC BY-SA 3.0"
- board text removed: "Yamaha SY99 8MB SRAM Expansion Wohmart.COM License: CC BY-SA 3.0"
