File: SY99_8MBEX.sch (KiCad schematic (older format))
At the start: 29 parts, among them J1 Conn_01x02, J2 Conn_02x20_Odd_Even, J3 Conn_01x14, J4 Conn_02x20_Odd_Even, U1 74ALVC164245DGG,51, U10 TXB0108PWR, U2 74ALVC164245DGG,51, U3 AZ1117EH-3.3TRG1, U4 SN74LVC1G97DBVR, U5 SN74LVC1G97DBVR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

Commit message: Version 1.1
Parts:
- removed J3: Conn_01x14, Pin_Headers:Pin_Header_Straight_1x14_Pitch2.54mm, symbol Conn_01x14
- removed U10, U9: TXB0108PWR, TXB0108PWR:TSSOP20, symbol TXB0108PWR
- added C11, C12, C13, C14, C15, C16, C17, C18: 100n, Capacitors_SMD:C_0805_HandSoldering, symbol C
- added J3: Conn_01x12_Male, Pin_Headers:Pin_Header_Straight_1x12_Pitch2.54mm, symbol Conn_01x12_Male
- added R3: 3k3, Resistors_SMD:R_0805_HandSoldering, symbol R
- added TP1: VRAM, Connectors:PINTST, symbol TEST
- added TP2: ~IC, Connectors:PINTST, symbol TEST
- added TP3: ~OE, Connectors:PINTST, symbol TEST
- added TP4: MSBW, Connectors:PINTST, symbol TEST
- added TP5: LSBW, Connectors:PINTST, symbol TEST
- added U9: SN74LVCH16T245, SN74LVCH16T245:TSSOP48, symbol SN74LVCH16T245
- C1, C2, C3: footprint Capacitors_Tantalum_SMD:CP_Tantalum_Case-B_EIA-3528-21_Reflow -> Capacitors_Tantalum_SMD:CP_Tantalum_Case-A_EIA-3216-18_Reflow
- C10, C6, C7, C8, C9: value 0.1u -> 100n
- D1, D2: footprint digikey-footprints:LED_5mm_Radial -> LEDs:LED_D5.0mm
- J2: footprint Pin_Headers:Pin_Header_Straight_2x20_Pitch2.54mm_SMD -> SY99:Socket_Strip_Straight_2x20_Pitch2.54mm_10.30Wide_SMD
- J4: footprint SY99:Socket_Strip_Straight_2x20_Pitch2.54mm_10.30Wide_SMD -> SY99:Pin_Header_Straight_2x20_Pitch2.54mm_10.30Wide_SMD
- R1: value 220R -> 1K; footprint Resistors_SMD:R_1210_HandSoldering -> Resistors_SMD:R_0805_HandSoldering
- R2: value 150R -> 1K; footprint Resistors_SMD:R_1210_HandSoldering -> Resistors_SMD:R_0805_HandSoldering
Connections:
- net labels added: CST
- wire segments 289 -> 310
- no-connect marks 17 -> 2
Other:
- note added: "N.B. J3 8-12 connect to\n10-14 on Molex 51004\n8-9 on Molex NC"
- moved on the sheet: C4, C5, D1, D2, R1, R2
